File: Hardware/Lipo_Charger_Basic.sch (EAGLE design)
At the start: 16 parts, among them U1 MCP73831

Commit message: Fixed silk issue, changed rev #'s for reds
Other:
- note added: "V10"
- note removed: "V01"
Changed lines of the file:
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@@
 <?xml version="1.0" encoding="utf-8"?>
 <!DOCTYPE eagle SYSTEM "eagle.dtd">
-<eagle version="6.4">
+<eagle version="7.2.0">
 <drawing>
 <settings>
@@
 <text x="58.674" y="123.952" size="1.778" layer="97">microUSB</text>
 <text x="148.59" y="7.112" size="2.54" layer="94">Revised by: Patrick Alberts</text>
-<text x="236.22" y="7.62" size="2.54" layer="94">V01</text>
+<text x="236.22" y="7.62" size="2.54" layer="94">V10</text>
 <text x="147.32" y="137.16" size="1.778" layer="97">Lipo Battery</text>
 </plain>
